File: mcu.kicad_sch (KiCad schematic)
At the start: 14 parts, among them SW1 SW_Push, U1 ATmega328P-A, Y1 16MHz

Commit message: Add files via upload
Parts:
- Y1: footprint Connector_PinHeader_2.54mm:PinHeader_1x16_P2.54mm_Vertical -> Crystal:Crystal_SMD_2016-4Pin_2.0x1.6mm
Changed lines of the file:
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@@
 			)
 		)
-		(property "Footprint" "Connector_PinHeader_2.54mm:PinHeader_1x16_P2.54mm_Vertical"
+		(property "Footprint" "Crystal:Crystal_SMD_2016-4Pin_2.0x1.6mm"
 			(at 213.36 101.6 0)
 			(effects
