File: peripherals .kicad_sch (KiCad schematic)
At the start: 3 parts, among them J2 Conn_01x16_Female, J3 Conn_01x16_Socket, J6 ICSP

Commit message: Add files via upload
Parts:
- J3: value Conn_01x16_Socket -> Conn_01x16_Female
Changed lines of the file:
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@@
 			)
 		)
-		(property "Value" "Conn_01x16_Socket"
+		(property "Value" "Conn_01x16_Female"
 			(at 97.79 45.72 0)
 			(effects
