File: SoCET Project.kicad_pcb (KiCad board)
At the start: 2 copper layers, 45 parts, among them J1 USB_C_Receptacle_USB2.0, J2 Conn_01x16_Female, J3 Conn_01x16_Socket, J6 ICSP, SW1 SW_Push, U1 ATmega328P-A, U2 LM1117DT-ADJ, U3 FT232RL, Y1 16MHz

Commit message: Add files via upload
Parts:
- J3: value Conn_01x16_Socket -> Conn_01x16_Female
- Y1: footprint Connector_PinHeader_2.54mm:PinHeader_1x16_P2.54mm_Vertical -> Crystal:Crystal_SMD_2016-4Pin_2.0x1.6mm
- moved R7 96.8 mm to (88.2, 87.0), turned to 0 degrees
- moved R5 91.5 mm to (88.2, 85.8), turned to 0 degrees
- moved C13 80.6 mm to (103.5, 94.8), turned to 0 degrees
- moved J2 77.5 mm to (160.3, 115.8)
- moved C12 74.1 mm to (110.2, 83.4)
- moved C15 72.6 mm to (90.2, 107.5), turned to -90 degrees
- moved D6 67.9 mm to (115.2, 97.5), turned to 90 degrees
- moved D5 67.8 mm to (113.2, 97.5)
- moved R11 65.8 mm to (113.2, 95.3)
- moved R12 65.7 mm to (115.2, 95.4)
- moved R8 61.0 mm to (90.5, 87.0), turned to 0 degrees
- moved R6 58.3 mm to (90.5, 85.8), turned to 0 degrees
- moved R10 56.2 mm to (94.5, 92.9), turned to 0 degrees
- moved R4 53.4 mm to (139.5, 99.8), turned to -90 degrees
- moved R3 53.1 mm to (137.9, 99.3), turned to 0 degrees
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Routing:
- net +3.3V: track 0.00 -> 113.2 mm, vias 0 -> 4
- net EX_RST: track 0.00 -> 92.7 mm, vias 0 -> 1
- net PWRU_IN: track 0.00 -> 76.4 mm, vias 0 -> 1
- net Net-(U2-ADJ): track 0.00 -> 75.0 mm
- net USART.TXD: track 0.00 -> 64.8 mm, vias 0 -> 1
- net USART.RXD: track 0.00 -> 59.6 mm
- net GPIO_C3: track 0.00 -> 55.2 mm, vias 0 -> 1
- net GND: track 0.00 -> 53.4 mm, vias 0 -> 33
- net GPIO_B1: track 0.00 -> 51.9 mm, vias 0 -> 1
- net GPIO_B0: track 0.00 -> 51.6 mm
- net Net-(C10-Pad1): track 0.00 -> 49.8 mm, vias 0 -> 2
- net GPIO_C2: track 0.00 -> 47.6 mm, vias 0 -> 1
- net GPIO_D7: track 0.00 -> 45.6 mm
- net GPIO_C5: track 0.00 -> 40.1 mm
- net USBC_D.N: track 0.00 -> 39.4 mm, vias 0 -> 2
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- added copper zone on B.Cu, net +5V
- added copper zone on F.Cu, net +5V
- added copper zone on B.Cu, net GND
- added copper zone on F.Cu, net GND
Other:
- board outline added: 80.5 x 48.7 mm
- board text added: "+3.3V"
- board text added: "+5.0V"
- board text added: "Aryan"
- board text added: "EX_IN"
- board text added: "GND"
- board text added: "ICSP"
- board text added: "IO_B0"
- board text added: "IO_B1"
- board text added: "IO_C0"
- board text added: "IO_C1"
- board text added: "IO_C2"
- board text added: "IO_C3"
- board text added: "IO_C4"
- board text added: "IO_C5"
- board text added: "IO_D2"
- board text added: "IO_D3"
- board text added: "IO_D4"
- board text added: "IO_D5"
- board text added: "IO_D6"
- board text added: "IO_D7"
- board text added: "MISO"
- board text added: "MOSI"
- board text added: "RST"
- board text added: "RXD"
- board text added: "SDA"
- board text added: "SS"
- board text added: "SoCET"
- board text added: "TXD"
- board text added: "X"

Commit message: Add files via upload
Completed SCH and DSG
Connections:
- D1 pad 2: USBC_D.P -> USBC_D.N
- D2 pad 2: USBC_D.N -> USBC_D.P
- U3 pad 15: USBC_D.P -> USBC_D.N
- U3 pad 16: USBC_D.N -> USBC_D.P
Routing:
- net SPI.MISO: track 29.7 -> 53.2 mm, vias 0 -> 2
- net GPIO_B1: track 51.9 -> 65.2 mm, vias 1 -> 2
- net +5V: track 0.00 -> 7.10 mm
- net USBC_D.P: track 36.8 -> 42.2 mm, vias 2 -> 0
- net EX_OSC2: track 34.9 -> 38.6 mm, vias 1 -> 4
- net USBC_D.N: track 39.4 -> 41.4 mm, vias 2 -> 0
- net Net-(U3-3V3OUT): track 5.64 -> 7.42 mm
- net Net-(J1-CC2): track 21.3 -> 23.0 mm, vias 1 -> 4
- net (no net): track 1.40 -> 0.00 mm
- net EX_OSC1: track 19.6 -> 20.9 mm, vias 1 -> 2
- net GND: track 53.4 -> 54.6 mm
- net Net-(C10-Pad1): track 49.8 -> 50.6 mm, vias 2 -> 4
- net EX_RST: track 92.7 -> 93.3 mm, vias 1 -> 2
- net GPIO_C2: track 47.6 -> 48.2 mm, vias 1 -> 2
- net GPIO_C3: track 55.2 -> 55.8 mm, vias 1 -> 2
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- removed copper zone on B.Cu, net +5V
- removed copper zone on F.Cu, net GND
Other:
- board size 80.5 x 48.7 mm -> 80.9 x 49.7 mm
