File: psu.kicad_sch (KiCad schematic)
At the start: 19 parts, among them J1 USB_C_Receptacle_USB2.0, U2 LM1117DT-ADJ

Commit message: Add files via upload
Completed SCH and DSG
Connections:
- net GND: now also D2.2 (A2); no longer D2.1 (A1)
- net USBC_D.N: now also D2.1 (A1); no longer D2.2 (A2)
Other:
- moved on the sheet: D2
Changed lines of the file:
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@@
 	(symbol
 		(lib_id "Diode:ESD9B5.0ST5G")
-		(at 83.82 93.98 90)
+		(at 83.82 93.98 270)
 		(unit 1)
 		(exclude_from_sim no)
@@
 					(size 1.27 1.27)
 				)
-				(justify right)
+				(justify left)
 			)
 		)
@@
 					(size 1.27 1.27)
 				)
-				(justify right)
+				(justify left)
 			)
 		)
